File: kicad/qlp-22/qlp-22_Mk1_rev0/qlp-22_Mk1_rev0.kicad_pcb (KiCad board)
At the start: 2 copper layers, 24 parts

Commit message: Begins restructuring of qlp-22 to matrix layout
Parts:
- added REF**: 1N4148, ScottoKeebs_Components:Diode_DO-35, F.Cu at (241.4, 200.2)
- added REF**: 1N4148, ScottoKeebs_Components:Diode_DO-35, F.Cu at (241.4, 137.8)
- added REF**: 1N4148, ScottoKeebs_Components:Diode_DO-35, F.Cu at (261.4, 137.8)
- added REF**: 1N4148, ScottoKeebs_Components:Diode_DO-35, F.Cu at (221.4, 160.2)
- added REF**: 1N4148, ScottoKeebs_Components:Diode_DO-35, F.Cu at (321.2, 160.2)
- added REF**: 1N4148, ScottoKeebs_Components:Diode_DO-35, F.Cu at (241.4, 160.2)
- added REF**: 1N4148, ScottoKeebs_Components:Diode_DO-35, F.Cu at (261.4, 160.2)
- added REF**: 1N4148, ScottoKeebs_Components:Diode_DO-35, F.Cu at (221.4, 200.2)
- added REF**: 1N4148, ScottoKeebs_Components:Diode_DO-35, F.Cu at (281.4, 160.2)
- added REF**: 1N4148, ScottoKeebs_Components:Diode_DO-35, F.Cu at (264.6, 45.2)
- added REF**: 1N4148, ScottoKeebs_Components:Diode_DO-35, F.Cu at (301.4, 160.2)
- added REF**: 1N4148, ScottoKeebs_Components:Diode_DO-35, F.Cu at (201.4, 200.2)
- moved REF** 70.0 mm to (110.4, 47.7), turned to 30 degrees
- moved REF** 65.8 mm to (329.0, 171.2), turned to 90 degrees
- moved REF** 60.0 mm to (120.4, 65.0), turned to -60 degrees
- moved REF** 55.7 mm to (309.0, 171.2), turned to 0 degrees
- moved REF** 50.2 mm to (130.4, 82.3), turned to -60 degrees
- moved REF** 46.2 mm to (115.8, 137.0), turned to 30 degrees
- moved REF** 45.8 mm to (289.0, 171.2), turned to 0 degrees
- moved REF** 41.4 mm to (249.0, 211.3), turned to 90 degrees
- moved REF** 41.2 mm to (125.8, 154.3), turned to 30 degrees
- moved REF** 40.6 mm to (140.4, 99.6), turned to -60 degrees
- moved REF** 38.3 mm to (135.8, 171.6), turned to 30 degrees
- moved REF** 37.2 mm to (159.9, 88.4), turned to 30 degrees
- moved REF** 36.7 mm to (229.0, 211.3), turned to 90 degrees
- moved REF** 36.0 mm to (269.0, 171.2), turned to 0 degrees
- moved REF** 34.5 mm to (209.0, 211.2), turned to 90 degrees
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Routing:
- net (no net): track 3182.8 -> 1029.7 mm

Commit message: Continues traces for matrix qlp-22 layout
Parts:
- removed the REF** at (264.6, 45.2)
- added REF**: 1N4148, ScottoKeebs_Components:Diode_DO-35, F.Cu at (170.2, 124.7)
- added REF**: 1N4148, ScottoKeebs_Components:Diode_DO-35, F.Cu at (89.7, 104.2)
- added REF**: 1N4148, ScottoKeebs_Components:Diode_DO-35, F.Cu at (152.9, 114.7)
- added REF**: 1N4148, ScottoKeebs_Components:Diode_DO-35, F.Cu at (173.6, 198.8)
- added REF**: 1N4148, ScottoKeebs_Components:Diode_DO-35, F.Cu at (139.0, 178.8)
- added REF**: 1N4148, ScottoKeebs_Components:Diode_DO-35, F.Cu at (124.4, 124.2)
- added REF**: 1N4148, ScottoKeebs_Components:Diode_DO-35, F.Cu at (159.0, 144.2)
- added REF**: 1N4148, ScottoKeebs_Components:Diode_DO-35, F.Cu at (141.7, 134.2)
- added REF**: 1N4148, ScottoKeebs_Components:Diode_DO-35, F.Cu at (176.3, 154.2)
- added REF**: 1N4148, ScottoKeebs_Components:Diode_DO-35, F.Cu at (156.3, 188.8)
- added REF**: 1N4148, ScottoKeebs_Components:Diode_DO-35, F.Cu at (107.0, 114.2)
- moved REF** 72.6 mm to (90.5, 117.5), turned to 60 degrees
- moved REF** 63.8 mm to (107.8, 127.5), turned to -30 degrees
- moved REF** 60.2 mm to (139.8, 192.2), turned to 60 degrees
- moved REF** 57.2 mm to (157.1, 202.2), turned to 60 degrees
- moved REF** 56.3 mm to (340.2, 116.0), turned to 120 degrees
- moved REF** 56.0 mm to (174.4, 212.2), turned to 60 degrees
- moved REF** 55.5 mm to (125.1, 137.5), turned to -30 degrees
- moved REF** 50.3 mm to (328.0, 110.4), turned to 30 degrees
- moved REF** 47.9 mm to (142.5, 147.5), turned to -30 degrees
- moved REF** 47.3 mm to (256.3, 210.7), turned to 120 degrees
- moved REF** 47.3 mm to (322.9, 126.0), turned to 30 degrees
- moved REF** 46.7 mm to (290.9, 190.7), turned to 120 degrees
- moved REF** 45.9 mm to (273.6, 200.7), turned to 120 degrees
- moved REF** 43.1 mm to (244.2, 205.0), turned to 30 degrees
- moved REF** 41.6 mm to (159.8, 157.5), turned to -30 degrees
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Routing:
- net (no net): track 1029.7 -> 2721.9 mm

Commit message: Adds row traces and comments for additional components
Parts:
- added REF**: Pin_D0.9mm_L10.0mm_W2.4mm_FlatFork, Connector_Pin:Pin_D0.9mm_L10.0mm_W2.4mm_FlatFork, F.Cu at (201.2, 129.9)
- added REF**: Pin_D0.9mm_L10.0mm_W2.4mm_FlatFork, Connector_Pin:Pin_D0.9mm_L10.0mm_W2.4mm_FlatFork, F.Cu at (201.2, 127.3)
- added REF**: Pin_D0.9mm_L10.0mm_W2.4mm_FlatFork, Connector_Pin:Pin_D0.9mm_L10.0mm_W2.4mm_FlatFork, F.Cu at (201.2, 132.5)
- moved REF** 14.6 mm to (161.7, 158.6)
- moved REF** 14.6 mm to (330.6, 124.8)
- moved REF** 14.6 mm to (244.2, 174.7)
- moved REF** 14.6 mm to (92.4, 118.6)
- moved REF** 14.6 mm to (159.8, 216.6)
- moved REF** 14.6 mm to (110.5, 141.9)
- moved REF** 14.6 mm to (267.6, 135.2)
- moved REF** 14.6 mm to (93.2, 131.9)
- moved REF** 14.6 mm to (250.2, 145.2)
- moved REF** 14.6 mm to (162.4, 171.9)
- moved REF** 14.6 mm to (176.3, 213.2)
- moved REF** 14.6 mm to (144.3, 148.6)
- moved REF** 14.6 mm to (177.1, 226.6)
- moved REF** 14.6 mm to (246.9, 219.4)
- moved REF** 14.6 mm to (273.6, 170.4)
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Routing:
- net (no net): track 2721.9 -> 2955.5 mm
Other:
- board text added: "Break out other I2C bus"
- board text added: "break out debug"
- board text added: "wire to left side"

Commit message: Adds reset button, breakouts for uart, i2c1 and debug
Parts:
- removed the REF** at (201.2, 129.9)
- removed the REF** at (201.2, 127.3)
- removed the REF** at (201.2, 132.5)
- added REF**: PinHeader_1x03_P2.54mm_Vertical, Connector_PinHeader_2.54mm:PinHeader_1x03_P2.54mm_Vertical, F.Cu at (200.7, 140.6)
- added REF**: PinHeader_1x03_P2.54mm_Vertical, Connector_PinHeader_2.54mm:PinHeader_1x03_P2.54mm_Vertical, F.Cu at (218.1, 185.5)
- added REF**: PinHeader_1x04_P2.54mm_Vertical, Connector_PinHeader_2.54mm:PinHeader_1x04_P2.54mm_Vertical, F.Cu at (198.9, 157.5)
- added REF**: SW_SPST_Omron_B3FS-101xP, Button_Switch_SMD:SW_SPST_Omron_B3FS-101xP, F.Cu at (239.1, 152.5)
- moved REF** 4.40 mm to (261.0, 229.0)
- moved REF** 4.40 mm to (248.9, 223.3)
- moved REF** 4.40 mm to (178.4, 217.1)
- moved REF** 4.40 mm to (293.0, 164.3)
- moved REF** 4.40 mm to (280.9, 158.6)
- moved REF** 4.40 mm to (179.1, 230.5)
- moved REF** 4.40 mm to (258.3, 184.3)
- moved REF** 4.40 mm to (332.7, 128.7)
- moved REF** 4.40 mm to (315.5, 138.6)
- moved REF** 4.40 mm to (246.2, 178.6)
- moved REF** 4.40 mm to (161.0, 207.1)
- moved REF** 4.40 mm to (269.6, 139.1)
- moved REF** 4.40 mm to (281.7, 144.8)
- moved REF** 4.40 mm to (181.8, 185.8)
- moved REF** 4.40 mm to (310.3, 154.3)
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Routing:
- net (no net): track 2955.5 -> 3241.2 mm
Other:
- board text added: "TODO: wrap rows on bottom"
- board text removed: "Break out other I2C bus"
- board text removed: "break out debug"
- board text removed: "wire to left side"

Commit message: Reworks row traces and pin breakouts for qlp-22
Parts:
- moved REF** 18.9 mm to (258.7, 195.9)
- moved REF** 18.9 mm to (308.0, 121.3)
- moved REF** 18.9 mm to (87.7, 118.5)
- moved REF** 18.9 mm to (174.3, 168.5)
- moved REF** 18.9 mm to (262.1, 121.8)
- moved REF** 18.9 mm to (250.8, 167.0)
- moved REF** 18.9 mm to (153.5, 189.8)
- moved REF** 18.9 mm to (273.3, 141.3)
- moved REF** 18.9 mm to (193.1, 123.3)
- moved REF** 18.9 mm to (270.8, 201.6)
- moved REF** 18.9 mm to (210.6, 168.1)
- moved REF** 18.9 mm to (302.8, 137.0)
- moved REF** 18.9 mm to (276.0, 185.9)
- moved REF** 18.9 mm to (137.0, 193.1)
- moved REF** 18.9 mm to (173.5, 155.1)
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Routing:
- net (no net): track 3241.2 -> 4007.1 mm
Other:
- board text removed: "TODO: wrap rows on bottom"

Commit message: Revises left hand centering back to original location
Parts:
- moved REF** 4.09 mm to (108.6, 126.5)
- moved REF** 4.09 mm to (171.0, 123.7)
- moved REF** 4.09 mm to (174.4, 197.8)
- moved REF** 4.09 mm to (125.9, 136.5)
- moved REF** 4.09 mm to (171.8, 137.0)
- moved REF** 4.09 mm to (177.1, 153.2)
- moved REF** 4.09 mm to (140.5, 191.1)
- moved REF** 4.09 mm to (175.2, 211.1)
- moved REF** 4.09 mm to (160.5, 156.5)
- moved REF** 4.09 mm to (157.1, 187.8)
- moved REF** 4.09 mm to (159.8, 143.2)
- moved REF** 4.09 mm to (125.1, 123.2)
- moved REF** 4.09 mm to (91.3, 116.5)
- moved REF** 4.09 mm to (143.2, 146.5)
- moved REF** 4.09 mm to (107.8, 113.2)
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Routing:
- net (no net): track 4007.1 -> 3889.9 mm

Commit message: Aligns f.Cu for left half of qpl-22
Parts:
- moved REF** 71.7 mm to (329.3, 187.4), turned to 90 degrees
- moved REF** 65.8 mm to (321.5, 176.4), turned to 0 degrees
- moved REF** 62.3 mm to (309.3, 187.4), turned to 0 degrees
- moved REF** 59.8 mm to (120.0, 51.2), turned to -60 degrees
- moved REF** 58.0 mm to (114.0, 63.2), turned to 30 degrees
- moved REF** 56.3 mm to (301.7, 176.4), turned to 0 degrees
- moved REF** 54.9 mm to (249.3, 227.4), turned to 90 degrees
- moved REF** 53.4 mm to (289.3, 187.4), turned to 0 degrees
- moved REF** 51.2 mm to (229.3, 227.4), turned to 90 degrees
- moved REF** 49.9 mm to (130.0, 68.5), turned to -60 degrees
- moved REF** 49.4 mm to (209.3, 227.4), turned to 90 degrees
- moved REF** 48.6 mm to (124.0, 80.5), turned to -60 degrees
- moved REF** 48.1 mm to (241.7, 216.4), turned to 0 degrees
- moved REF** 47.1 mm to (281.7, 176.4), turned to 0 degrees
- moved REF** 44.9 mm to (269.3, 187.4), turned to 0 degrees
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Routing:
- net (no net): track 3889.9 -> 3888.8 mm
Other:
- board text added: "TODO work on spacing the f.Cu on this right half"

Commit message: Finishes revisions to f.Cu on qlp-22
Parts:
- moved REF** 72.0 mm to (86.3, 114.9), turned to -30 degrees
- moved REF** 70.4 mm to (87.1, 128.2), turned to 60 degrees
- moved REF** 62.2 mm to (103.6, 124.9), turned to -30 degrees
- moved REF** 61.0 mm to (104.4, 138.2), turned to -30 degrees
- moved REF** 59.6 mm to (335.7, 128.2), turned to 120 degrees
- moved REF** 53.9 mm to (323.4, 122.6), turned to 30 degrees
- moved REF** 53.2 mm to (136.4, 202.8), turned to 60 degrees
- moved REF** 52.6 mm to (121.0, 134.9), turned to -30 degrees
- moved REF** 51.9 mm to (121.8, 148.2), turned to -30 degrees
- moved REF** 50.1 mm to (318.4, 138.2), turned to 30 degrees
- moved REF** 50.1 mm to (135.6, 189.5), turned to -30 degrees
- moved REF** 49.5 mm to (153.7, 212.8), turned to 60 degrees
- moved REF** 47.7 mm to (171.0, 222.8), turned to 60 degrees
- moved REF** 45.2 mm to (152.9, 199.5), turned to -30 degrees
- moved REF** 44.5 mm to (286.4, 202.8), turned to 120 degrees
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Routing:
- net (no net): track 3888.8 -> 3891.0 mm
Other:
- board text removed: "TODO work on spacing the f.Cu on this right half"
