File: kicad/qlp-22/qlp-22_Mk1_rev0/qlp-22_Mk1_rev0.kicad_pcb (KiCad board)
At the start: 2 copper layers, 50 parts

Commit message: Aligns b.Cu layer of qlp-22
Parts:
- moved REF** 7.45 mm to (155.0, 175.5)
- moved REF** 7.45 mm to (238.3, 224.4)
- moved REF** 7.45 mm to (119.6, 142.2)
- moved REF** 7.45 mm to (166.2, 156.0)
- moved REF** 7.45 mm to (120.4, 155.5)
- moved REF** 7.45 mm to (148.9, 146.0)
- moved REF** 7.45 mm to (304.9, 139.8)
- moved REF** 7.45 mm to (136.9, 152.2)
- moved REF** 7.45 mm to (84.9, 122.2)
- moved REF** 7.45 mm to (285.0, 210.1)
- moved REF** 7.45 mm to (322.0, 129.9)
- moved REF** 7.45 mm to (102.2, 132.2)
- moved REF** 7.45 mm to (271.1, 146.0)
- moved REF** 7.45 mm to (247.7, 185.5)
- moved REF** 7.45 mm to (267.7, 220.1)
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Routing:
- net (no net): track 3891.0 -> 3884.7 mm

Commit message: Creates initial pcb edge outline for qlp-22
Parts:
- moved REF** 30.9 mm to (275.7, 212.5)
- moved REF** 30.9 mm to (191.6, 138.3)
- moved REF** 30.9 mm to (111.1, 117.8)
- moved REF** 30.9 mm to (310.3, 192.5)
- moved REF** 30.9 mm to (278.2, 152.1)
- moved REF** 30.9 mm to (325.0, 137.8)
- moved REF** 30.9 mm to (312.9, 132.1)
- moved REF** 30.9 mm to (195.0, 212.5)
- moved REF** 30.9 mm to (342.3, 127.8)
- moved REF** 30.9 mm to (159.5, 179.1)
- moved REF** 30.9 mm to (290.3, 157.8)
- moved REF** 30.9 mm to (179.5, 144.5)
- moved REF** 30.9 mm to (176.9, 189.1)
- moved REF** 30.9 mm to (194.2, 199.1)
- moved REF** 30.9 mm to (330.2, 122.1)
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Other:
- board outline added: 294.5 x 144.3 mm

Commit message: Adds rounded edges and initial mounting holes to qlp-22
Parts:
- moved REF** 16.6 mm to (185.5, 140.8)
- moved REF** 16.6 mm to (230.0, 195.1)
- moved REF** 16.6 mm to (324.9, 137.9)
- moved REF** 16.6 mm to (175.1, 173.6)
- moved REF** 16.6 mm to (174.3, 160.3)
- moved REF** 16.6 mm to (293.0, 202.5)
- moved REF** 16.6 mm to (157.7, 163.6)
- moved REF** 16.6 mm to (105.0, 120.3)
- moved REF** 16.6 mm to (192.4, 183.6)
- moved REF** 16.6 mm to (273.0, 167.9)
- moved REF** 16.6 mm to (302.4, 163.6)
- moved REF** 16.6 mm to (248.5, 151.8)
- moved REF** 16.6 mm to (105.8, 133.6)
- moved REF** 16.6 mm to (139.6, 140.3)
- moved REF** 16.6 mm to (270.4, 228.2)
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Routing:
- net (no net): track 3884.7 -> 3884.1 mm
Other:
- board size 294.5 x 144.3 mm -> 292.7 x 142.4 mm

Commit message: Begins silkscreening qlp-22
Parts:
- moved REF** 26.0 mm to (98.1, 95.1)
- moved REF** 26.0 mm to (182.0, 189.8)
- moved REF** 26.0 mm to (298.2, 183.1)
- moved REF** 26.0 mm to (150.1, 125.1)
- moved REF** 26.0 mm to (268.8, 187.4)
- moved REF** 26.0 mm to (133.6, 128.5)
- moved REF** 26.0 mm to (201.4, 131.6)
- moved REF** 26.0 mm to (254.9, 123.3)
- moved REF** 26.0 mm to (179.5, 129.0)
- moved REF** 26.0 mm to (98.9, 108.5)
- moved REF** 26.0 mm to (283.4, 132.7)
- moved REF** 26.0 mm to (318.1, 112.7)
- moved REF** 26.0 mm to (284.3, 119.0)
- moved REF** 26.0 mm to (161.3, 105.6)
- moved REF** 26.0 mm to (115.4, 105.1)
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Other:
- board size 292.7 x 142.4 mm -> 292.7 x 142.5 mm
- board text added: "10-2023"
- board text added: "HAMLUND MFG."
- board text added: "Mk I"
- board text added: "QLP-22"
- board text added: "QLP-22-MK.1-REV.0"
- board text added: "Qwerty Linear Paginated Keyboard"
- board text added: "prototype revision 0 2023"

Commit message: Adds front qlp-22 silkscreen for all switches and diodes
Parts:
- renumbered REF** to D0:10, REF** to D0:3, REF** to D0:4, REF** to D0:9, REF** to D1:0, REF** to D1:1, REF** to D1:10, REF** to D1:11, REF** to D1:12, REF** to D1:13, REF** to D1:2, REF** to D1:3, REF** to D1:4, REF** to D1:5, REF** to D1:8, REF** to D1:9, REF** to D2:4, REF** to D2:5, REF** to D2:6, REF** to D2:7, REF** to D2:8, REF** to D2:9, REF** to S0:10, REF** to S0:3, REF** to S0:4, REF** to S0:9, REF** to S1:0, REF** to S1:1, REF** to S1:10, REF** to S1:11, REF** to S1:12, REF** to S1:13, REF** to S1:2, REF** to S1:3, REF** to S1:4, REF** to S1:5, REF** to S1:8, REF** to S1:9, REF** to S2:4, REF** to S2:5, REF** to S2:6, REF** to S2:7, REF** to S2:8, REF** to S2:9

Commit message: Revises and labels front and back qlp-22 silkscreen
Parts:
- moved S0:10 7.32 mm to (277.6, 121.9)
- moved D2:8 7.32 mm to (262.1, 190.4)
- moved D0:4 7.32 mm to (172.0, 118.6)
- moved D1:8 7.32 mm to (242.1, 155.7)
- moved D0:9 7.32 mm to (248.2, 126.2)
- moved S1:10 7.32 mm to (288.8, 141.4)
- moved S1:3 7.32 mm to (144.2, 141.4)
- moved S1:8 7.32 mm to (254.2, 161.4)
- moved S2:8 7.32 mm to (274.2, 196.1)
- moved DEBUG 7.32 mm to (214.0, 162.6)
- moved D0:10 7.32 mm to (265.5, 116.2)
- moved S2:7 7.32 mm to (256.9, 206.1)
- moved D2:7 7.32 mm to (244.8, 200.4)
- moved S1:4 7.32 mm to (161.5, 151.4)
- moved S2:5 7.32 mm to (158.8, 196.1)
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- renumbered REF** to DEBUG, REF** to I2C1, REF** to RESET, REF** to UART0
Routing:
- net (no net): track 3884.1 -> 3882.7 mm
Other:
- board size 292.7 x 142.5 mm -> 292.7 x 142.4 mm
- board text added: "C0-GP3"
- board text added: "C1-GP4"
- board text added: "C10-GP22"
- board text added: "C11-GP26"
- board text added: "C12-GP27"
- board text added: "C13-GP28"
- board text added: "C2-GP6"
- board text added: "C3-GP7"
- board text added: "C4-GP12"
- board text added: "C5-GP13"
- board text added: "C6-GP14"
- board text added: "C7-GP16"
- board text added: "C8-GP17"
- board text added: "C9-GP21"
- board text added: "GND"
- board text added: "I2C-VCC"
- board text added: "I2C0"
- board text added: "I2C0-GND"
- board text added: "I2C0-SCL"
- board text added: "I2C0-SDA"
- board text added: "I2C1-GND"
- board text added: "I2C1-SCL"
- board text added: "I2C1-SDA"
- board text added: "JLCJLCJLCJLC"
- board text added: "OLED 128x64"
- board text added: "R0-GP20"
- board text added: "R1-GP19"
- board text added: "R2-GP18"
- board text added: "RX/GP1"
- board text added: "Raspberry Pi Pico"
- board text added: "S0:10"
- board text added: "S0:3"
- board text added: "S0:4"
- board text added: "S0:9"
- board text added: "S1:0"
- board text added: "S1:1"
- board text added: "S1:10"
- board text added: "S1:11"
- board text added: "S1:12"
- board text added: "S1:13"
- board text added: "S1:2"
- board text added: "S1:3"
- board text added: "S1:4"
- board text added: "S1:5"
- board text added: "S1:8"
- board text added: "S1:9"
- board text added: "S2:4"
- board text added: "S2:5"
- board text added: "S2:6"
- board text added: "S2:7"
- board text added: "S2:8"
- board text added: "S2:9"
- board text added: "SCL/GP11"
- board text added: "SCL/GP5"
- board text added: "SDA/GP10"
- board text added: "SDA/GP8"
- board text added: "SWCLK"
- board text added: "SWDIO"
- board text added: "TX/GP0"
- board text added: "UART0-G"
- board text added: "UART0-RX"
- board text added: "UART0-TX"
- board text added: "VCC/VSYS"
