File: kicad/qlp-22/qlp-22_Mk1_rev1/qlp-22_Mk1_rev1.kicad_pcb (KiCad board)
At the start: 2 copper layers, 14 parts

Commit message: Adds remaining footprints for qlp-22_Mk1_rev1 pcb
Parts:
- added REF**: 1N4148, ScottoKeebs_Components:Diode_DO-35, F.Cu at (207.6, 196.7)
- added REF**: OLED_128x64, ScottoKeebs_Components:OLED_128x64, F.Cu at (226.5, 159.2)
- added REF**: Choc_V1V2_1.25u, ScottoKeebs_Choc:Choc_V1V2_1.25u, F.Cu at (276.9, 177.4)
- added REF**: Choc_V1V2_1.00u, ScottoKeebs_Choc:Choc_V1V2_1.00u, F.Cu at (282.0, 133.0)
- added REF**: PinHeader_1x04_P2.54mm_Vertical, Connector_PinHeader_2.54mm:PinHeader_1x04_P2.54mm_Vertical, F.Cu at (209.0, 140.5)
- added REF** (x2): 1N4148, ScottoKeebs_Components:Diode_DO-35, F.Cu at (238.2, 199.0)
- added REF**: 1N4148, ScottoKeebs_Components:Diode_DO-35, F.Cu at (262.1, 147.8)
- added REF**: PinHeader_1x04_P2.54mm_Vertical, Connector_PinHeader_2.54mm:PinHeader_1x04_P2.54mm_Vertical, F.Cu at (484.0, 126.0)
- added REF**: 1N4148, ScottoKeebs_Components:Diode_DO-35, F.Cu at (84.6, 125.4)
- added REF**: Choc_V1V2_1.50u, ScottoKeebs_Choc:Choc_V1V2_1.50u, F.Cu at (360.6, 115.1)
- added REF**: 1N4148, ScottoKeebs_Components:Diode_DO-35, F.Cu at (298.0, 129.4)
- added REF**: 1N4148, ScottoKeebs_Components:Diode_DO-35, F.Cu at (266.9, 102.4)
- added REF**: PinHeader_1x03_P2.54mm_Vertical, Connector_PinHeader_2.54mm:PinHeader_1x03_P2.54mm_Vertical, F.Cu at (209.0, 103.5)
- added REF**: SW_SPST_Omron_B3FS-101xP, Button_Switch_SMD:SW_SPST_Omron_B3FS-101xP, F.Cu at (246.0, 114.0)
- added REF**: 1N4148, ScottoKeebs_Components:Diode_DO-35, F.Cu at (194.6, 177.1)
- added REF** (x2): 1N4148, ScottoKeebs_Components:Diode_DO-35, F.Cu at (342.7, 135.4)
- added REF**: 1N4148, ScottoKeebs_Components:Diode_DO-35, F.Cu at (430.0, 123.0)
- added REF**: 1N4148, ScottoKeebs_Components:Diode_DO-35, F.Cu at (163.6, 83.9)
- added REF**: Choc_V1V2_1.00u, ScottoKeebs_Choc:Choc_V1V2_1.00u, F.Cu at (261.5, 135.2)
- added REF**: Choc_V1V2_1.00u, ScottoKeebs_Choc:Choc_V1V2_1.00u, F.Cu at (317.9, 114.6)
- added REF**: 1N4148, ScottoKeebs_Components:Diode_DO-35, F.Cu at (127.3, 125.0)
- added REF**: SW_SPST_Omron_B3FS-101xP, Button_Switch_SMD:SW_SPST_Omron_B3FS-101xP, F.Cu at (461.0, 139.0)
- added REF**: PinHeader_1x03_P2.54mm_Vertical, Connector_PinHeader_2.54mm:PinHeader_1x03_P2.54mm_Vertical, F.Cu at (224.5, 155.0)
- added REF**: 1N4148, ScottoKeebs_Components:Diode_DO-35, F.Cu at (184.1, 144.5)
- added REF**: Choc_V1V2_1.25u, ScottoKeebs_Choc:Choc_V1V2_1.25u, F.Cu at (259.8, 189.0)
- added REF**: 1N4148, ScottoKeebs_Components:Diode_DO-35, F.Cu at (252.2, 179.0)
- added REF**: Choc_V1V2_1.00u, ScottoKeebs_Choc:Choc_V1V2_1.00u, F.Cu at (297.4, 116.8)
- added REF**: Raspberry_Pi_Pico, ScottoKeebs_MCU:Raspberry_Pi_Pico, F.Cu at (226.5, 125.2)
- added REF**: PinHeader_1x03_P2.54mm_Vertical, Connector_PinHeader_2.54mm:PinHeader_1x03_P2.54mm_Vertical, F.Cu at (461.0, 119.0)
- added REF**: 1N4148, ScottoKeebs_Components:Diode_DO-35, F.Cu at (147.8, 127.1)
- added REF**: Choc_V1V2_1.00u, ScottoKeebs_Choc:Choc_V1V2_1.00u, F.Cu at (341.8, 121.9)
- added REF**: 1N4148, ScottoKeebs_Components:Diode_DO-35, F.Cu at (176.9, 164.3)
- added REF**: Choc_V1V2_1.25u, ScottoKeebs_Choc:Choc_V1V2_1.25u, F.Cu at (274.3, 111.9)
- added REF**: 1N4148, ScottoKeebs_Components:Diode_DO-35, F.Cu at (282.2, 86.2)
- added REF**: 1N4148, ScottoKeebs_Components:Diode_DO-35, F.Cu at (269.6, 168.4)
- added REF**: 1N4148, ScottoKeebs_Components:Diode_DO-35, F.Cu at (318.5, 127.2)
- added REF**: Choc_V1V2_1.50u, ScottoKeebs_Choc:Choc_V1V2_1.50u, F.Cu at (246.1, 209.9)
- added REF**: 1N4148, ScottoKeebs_Components:Diode_DO-35, F.Cu at (103.1, 133.1)
- added REF**: Choc_V1V2_1.25u, ScottoKeebs_Choc:Choc_V1V2_1.25u, F.Cu at (289.7, 95.6)
- added REF**: 1N4148, ScottoKeebs_Components:Diode_DO-35, F.Cu at (163.6, 142.1)
- added REF**: 1N4148, ScottoKeebs_Components:Diode_DO-35, F.Cu at (282.3, 144.7)
- added REF**: 1N4148, ScottoKeebs_Components:Diode_DO-35, F.Cu at (361.2, 127.7)
- added REF**: 1N4148, ScottoKeebs_Components:Diode_DO-35, F.Cu at (179.3, 99.2)
- moved REF** 188.4 mm to (450.2, 94.5)
- moved REF** 188.4 mm to (449.2, 66.7)
- moved REF** 188.4 mm to (449.2, 38.5)
- moved REF** 93.1 mm to (206.8, 209.9), turned to 70 degrees
- moved REF** 92.0 mm to (178.9, 112.0), turned to 70 degrees
- moved REF** 88.8 mm to (163.3, 95.6), turned to 70 degrees
- moved REF** 88.2 mm to (193.2, 189.0), turned to 70 degrees
- moved REF** 87.3 mm to (171.0, 133.0), turned to 160 degrees
- moved REF** 85.4 mm to (191.5, 135.2), turned to 160 degrees
- moved REF** 83.7 mm to (155.6, 116.8), turned to 160 degrees
- moved REF** 82.4 mm to (176.1, 177.4), turned to 70 degrees
- moved REF** 77.3 mm to (135.1, 114.6), turned to 160 degrees
- moved REF** 68.6 mm to (111.2, 121.9), turned to 160 degrees
- moved REF** 63.5 mm to (92.4, 115.1), turned to 70 degrees

Commit message: Adds starts of row/col tracks and sets board outline
Parts:
- moved REF** 5.55 mm to (265.1, 165.3)
- moved REF** 5.55 mm to (277.4, 129.9)
- moved REF** 5.55 mm to (277.7, 83.0)
- moved REF** 5.55 mm to (241.6, 206.8)
- moved REF** 5.55 mm to (186.9, 132.0)
- moved REF** 5.55 mm to (479.4, 122.8)
- moved REF** 5.55 mm to (190.0, 173.9)
- moved REF** 5.55 mm to (221.9, 122.0)
- moved REF** 5.55 mm to (425.4, 119.8)
- moved REF** 5.55 mm to (158.8, 92.5)
- moved REF** 5.55 mm to (172.3, 161.1)
- moved REF** 5.55 mm to (445.6, 91.4)
- moved REF** 5.55 mm to (241.4, 110.8)
- moved REF** 5.55 mm to (256.9, 132.0)
- moved REF** 5.55 mm to (444.6, 63.6)
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Routing:
- net (no net): track 0.00 -> 1541.0 mm
Other:
- board outline added: 301 x 153 mm

Commit message: Places initial mounting holes
Parts:
- moved REF** 9.94 mm to (200.9, 109.6)
- moved REF** 3.69 mm to (274.2, 142.7)
- moved REF** 3.69 mm to (441.1, 64.7)
- moved REF** 3.69 mm to (119.3, 122.9)
- moved REF** 3.69 mm to (273.9, 131.0)
- moved REF** 3.69 mm to (168.0, 175.4)
- moved REF** 3.69 mm to (442.1, 92.5)
- moved REF** 3.69 mm to (253.4, 133.1)
- moved REF** 3.69 mm to (176.0, 142.5)
- moved REF** 3.69 mm to (266.2, 109.9)
- moved REF** 3.69 mm to (183.4, 133.1)
- moved REF** 3.69 mm to (218.4, 157.1)
- moved REF** 3.69 mm to (84.3, 113.0)
- moved REF** 3.69 mm to (127.0, 112.6)
- moved REF** 3.69 mm to (147.5, 114.8)
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Other:
- outline, holes or cut-outs redrawn

Commit message: Removes fCu dimensions, adds silkscreen to qlp-22_Mk1_rev1
Parts:
- removed the REF** at (475.9, 124.0)
- removed the REF** at (421.9, 121.0)
- removed the REF** at (452.9, 137.0)
- removed the REF** at (452.9, 117.0)
- removed the REF** at (442.1, 92.5)
- removed the REF** at (441.1, 36.5)
- removed the REF** at (441.1, 64.7)
- moved REF** 2.31 mm to (203.0, 108.6)
- moved REF** 2.31 mm to (188.6, 174.1)
- moved REF** 2.31 mm to (253.8, 186.0)
- moved REF** 2.31 mm to (105.2, 118.9)
- moved REF** 2.31 mm to (97.1, 130.1)
- moved REF** 2.31 mm to (220.5, 156.2)
- moved REF** 2.31 mm to (187.2, 186.0)
- moved REF** 2.31 mm to (218.5, 152.0)
- moved REF** 2.31 mm to (78.6, 122.4)
- moved REF** 2.31 mm to (157.6, 80.9)
- moved REF** 2.31 mm to (354.6, 112.0)
- moved REF** 2.31 mm to (260.9, 99.4)
- moved REF** 2.31 mm to (141.9, 124.1)
- moved REF** 2.31 mm to (312.5, 124.2)
- moved REF** 2.31 mm to (149.6, 113.8)
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Other:
- outline, holes or cut-outs redrawn

Commit message: Finalizes diode positions for qlp-22_Mk1_rev1
Parts:
- removed the REF** at (336.8, 132.4)
- removed the REF** at (232.2, 196.0)
- moved REF** 13.4 mm to (289.5, 139.5)
- moved REF** 13.2 mm to (325.4, 121.1)
- moved REF** 13.2 mm to (368.1, 121.6)
- moved REF** 13.2 mm to (304.9, 123.3)
- moved REF** 13.2 mm to (245.1, 192.9)
- moved REF** 13.2 mm to (269.0, 141.7)
- moved REF** 13.2 mm to (349.3, 128.4)
- moved REF** 13.2 mm to (258.7, 172.0)
- moved REF** 13.2 mm to (275.8, 160.5)
- moved REF** 13.2 mm to (288.6, 78.7)
- moved REF** 13.2 mm to (273.2, 94.9)
- moved REF** 13.2 mm to (110.1, 128.4)
- moved REF** 12.7 mm to (91.3, 121.6)
- moved REF** 12.7 mm to (134.1, 121.1)
- moved REF** 12.7 mm to (154.6, 123.3)
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Routing:
- net (no net): track 1541.0 -> 1154.3 mm
Other:
- outline, holes or cut-outs redrawn

Commit message: Adds more row wiring to right side
Parts:
- moved REF** 20.1 mm to (331.1, 137.0)
- moved REF** 20.1 mm to (77.4, 118.4)
- moved REF** 20.1 mm to (161.0, 100.9)
- moved REF** 20.1 mm to (148.3, 99.0)
- moved REF** 20.1 mm to (240.5, 180.6)
- moved REF** 20.1 mm to (349.9, 130.1)
- moved REF** 20.1 mm to (96.2, 125.2)
- moved REF** 20.1 mm to (161.1, 180.8)
- moved REF** 20.1 mm to (175.3, 178.0)
- moved REF** 20.1 mm to (211.5, 128.5)
- moved REF** 20.1 mm to (163.9, 115.3)
- moved REF** 20.1 mm to (136.3, 131.9)
- moved REF** 20.1 mm to (120.1, 118.0)
- moved REF** 20.1 mm to (194.0, 143.8)
- moved REF** 20.1 mm to (178.2, 192.3)
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Routing:
- net (no net): track 1154.3 -> 1415.5 mm

Commit message: Adds the row and column buses for qlp-22_Mk1_rev1
Parts:
- moved REF** 7.25 mm to (186.3, 217.9)
- moved REF** 7.25 mm to (225.6, 217.9)
- moved REF** 7.25 mm to (188.4, 148.4)
- moved REF** 7.25 mm to (158.3, 119.9)
- moved REF** 7.25 mm to (135.0, 124.7)
- moved REF** 7.25 mm to (340.0, 123.0)
- moved REF** 7.25 mm to (221.3, 206.1)
- moved REF** 7.25 mm to (253.7, 119.8)
- moved REF** 7.25 mm to (67.5, 134.8)
- moved REF** 7.25 mm to (90.6, 129.9)
- moved REF** 7.25 mm to (264.8, 91.9)
- moved REF** 7.25 mm to (301.6, 134.4)
- moved REF** 7.25 mm to (130.8, 136.5)
- moved REF** 7.25 mm to (71.8, 123.0)
- moved REF** 7.25 mm to (203.9, 163.0)
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Routing:
- net (no net): track 1415.5 -> 2520.0 mm
Other:
- outline, holes or cut-outs redrawn

Commit message: Adds majority of column hookups for qlp-22_Mk1_rev1
Parts:
- added REF**: MountingHole_2.2mm_M2, MountingHole:MountingHole_2.2mm_M2, F.Cu at (283.4, 182.3)
- moved REF** 45.0 mm to (225.9, 173.3)
- moved REF** 26.4 mm to (227.9, 148.3)
- moved REF** 20.5 mm to (191.9, 139.8), turned to 180 degrees
- moved REF** 19.4 mm to (191.9, 178.3), turned to 180 degrees
- moved REF** 18.5 mm to (243.9, 161.4)
- moved REF** 18.5 mm to (133.7, 154.8)
- moved REF** 18.5 mm to (189.2, 236.2)
- moved REF** 18.5 mm to (264.4, 159.3)
- moved REF** 18.5 mm to (142.8, 107.5)
- moved REF** 18.5 mm to (324.2, 148.1)
- moved REF** 18.5 mm to (279.8, 143.0)
- moved REF** 18.5 mm to (186.4, 221.8)
- moved REF** 18.5 mm to (343.0, 141.3)
- moved REF** 18.5 mm to (259.3, 203.7)
- moved REF** 18.5 mm to (158.5, 203.7)
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Routing:
- net (no net): track 2520.0 -> 4237.9 mm
