File: kicad/seok-38/seok-38_Mk1_rev0/seok-38_Mk1_rev0.kicad_pcb (KiCad board)
At the start: 2 copper layers, 84 parts

Commit message: Adds left half edgecuts for seok-38_Mk1_rev0
Parts:
- moved REF** 4.25 mm to (174.4, 140.4)
- moved REF** 4.25 mm to (146.5, 136.1)
- moved REF** 4.25 mm to (324.8, 127.6)
- moved REF** 4.25 mm to (318.0, 108.8)
- moved REF** 4.25 mm to (135.1, 131.4)
- moved REF** 4.25 mm to (328.1, 136.5)
- moved REF** 4.25 mm to (254.6, 110.0)
- moved REF** 4.25 mm to (163.6, 147.6)
- moved REF** 4.25 mm to (224.9, 203.8)
- moved REF** 4.25 mm to (268.3, 147.6)
- moved REF** 4.25 mm to (225.9, 153.4)
- moved REF** 4.25 mm to (226.9, 139.4)
- moved REF** 4.25 mm to (121.4, 110.4)
- moved REF** 4.25 mm to (181.2, 121.6)
- moved REF** 4.25 mm to (237.5, 121.6)
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Other:
- board outline added: 144.2 x 158 mm

Commit message: Completes the edge cuts for seok-38_Mk1_rev0
Parts:
- moved REF** 6.98 mm to (229.6, 145.8)
- moved REF** 6.98 mm to (283.1, 128.9)
- moved REF** 6.98 mm to (317.1, 105.3)
- moved REF** 6.98 mm to (173.2, 135.3)
- moved REF** 6.98 mm to (133.9, 126.3)
- moved REF** 6.98 mm to (267.7, 145.1)
- moved REF** 6.98 mm to (212.1, 173.8)
- moved REF** 6.98 mm to (227.6, 210.3)
- moved REF** 6.98 mm to (243.8, 137.9)
- moved REF** 6.98 mm to (179.6, 198.3)
- moved REF** 6.98 mm to (306.9, 135.7)
- moved REF** 6.98 mm to (89.4, 131.4)
- moved REF** 6.98 mm to (269.4, 91.3)
- moved REF** 6.98 mm to (289.9, 89.2)
- moved REF** 6.98 mm to (303.6, 126.8)
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Other:
- board size 144.2 x 158 mm -> 294.1 x 158 mm

Commit message: Adds the row wiring for seok-38_Mk1_rev0
Parts:
- removed the REF** at (228.6, 159.8)
- moved REF** 6.23 mm to (233.7, 124.4)
- moved REF** 6.23 mm to (266.1, 96.6)
- moved REF** 6.23 mm to (236.9, 133.3)
- moved REF** 6.23 mm to (144.3, 94.0)
- moved REF** 6.23 mm to (86.1, 136.7)
- moved REF** 6.23 mm to (250.6, 170.9)
- moved REF** 6.23 mm to (310.6, 101.7)
- moved REF** 6.23 mm to (134.5, 143.1)
- moved ? 6.23 mm to (262.9, 146.1)
- moved REF** 6.23 mm to (240.5, 143.2)
- moved ? 6.23 mm to (256.0, 127.3)
- moved REF** 6.23 mm to (238.0, 194.6)
- moved REF** 6.23 mm to (141.3, 124.3)
- moved REF** 6.23 mm to (243.8, 152.1)
- moved REF** 6.23 mm to (241.2, 203.6)
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Routing:
- net (no net): track 0.00 -> 2367.9 mm

Commit message: Adds column wiring to seok-38_Mk1_rev0
Parts:
- moved REF** 4.85 mm to (273.0, 128.0)
- moved REF** 4.85 mm to (247.6, 116.5)
- moved REF** 4.85 mm to (173.5, 125.4)
- moved REF** 4.85 mm to (177.4, 136.9)
- moved REF** 4.85 mm to (86.9, 151.9)
- moved REF** 4.85 mm to (110.8, 144.6)
- moved REF** 4.85 mm to (170.6, 155.7)
- moved REF** 4.85 mm to (266.2, 109.2)
- moved ? 4.85 mm to (259.7, 149.7)
- moved REF** 4.85 mm to (169.2, 195.7)
- moved REF** 4.85 mm to (74.9, 126.2)
- moved REF** 4.85 mm to (321.1, 142.9)
- moved REF** 4.85 mm to (146.7, 163.0)
- moved REF** 4.85 mm to (142.8, 151.5)
- moved REF** 4.85 mm to (156.4, 113.9)
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Routing:
- net (no net): track 2367.9 -> 3327.4 mm

Commit message: Completes row hookups for seok-38_Mk1_rev0
Parts:
- moved REF** 20.8 mm to (121.2, 94.9)
- moved REF** 20.8 mm to (163.9, 94.5)
- moved REF** 20.8 mm to (231.9, 208.8)
- moved REF** 20.8 mm to (307.9, 125.2)
- moved REF** 20.8 mm to (118.3, 125.2)
- moved REF** 20.8 mm to (259.4, 167.4)
- moved REF** 20.8 mm to (132.0, 87.6)
- moved REF** 20.8 mm to (304.7, 116.3)
- moved REF** 20.8 mm to (340.5, 97.9)
- moved REF** 20.8 mm to (150.3, 132.1)
- moved REF** 20.8 mm to (108.1, 94.9)
- moved REF** 20.8 mm to (174.2, 124.8)
- moved REF** 20.8 mm to (297.8, 97.5)
- moved REF** 20.8 mm to (97.3, 102.2)
- moved REF** 20.8 mm to (314.9, 86.0)
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Routing:
- net (no net): track 3327.4 -> 4177.6 mm, vias 0 -> 6
Other:
- board text added: "R0"
- board text added: "R1"
- board text added: "R2"
- board text added: "R3"

Commit message: Completes column hookups for seok-38_Mk1_rev0
Parts:
- added REF**: MountingHole_2.2mm_M2_ISO14580, MountingHole:MountingHole_2.2mm_M2_ISO14580, F.Cu at (187.8, 161.5)
- added REF**: MountingHole_2.2mm_M2_ISO14580, MountingHole:MountingHole_2.2mm_M2_ISO14580, F.Cu at (212.8, 201.5)
- added REF**: MountingHole_2.2mm_M2_ISO14580, MountingHole:MountingHole_2.2mm_M2_ISO14580, F.Cu at (91.9, 90.8)
- added REF**: MountingHole_2.2mm_M2_ISO14580, MountingHole:MountingHole_2.2mm_M2_ISO14580, F.Cu at (333.8, 90.8)
- added REF**: MountingHole_2.2mm_M2_ISO14580, MountingHole:MountingHole_2.2mm_M2_ISO14580, F.Cu at (237.8, 161.5)
- moved ? 6.88 mm to (260.1, 104.7)
- moved REF** 6.88 mm to (134.6, 109.0)
- moved REF** 6.88 mm to (264.9, 117.9)
- moved REF** 6.88 mm to (131.7, 80.8)
- moved REF** 6.88 mm to (82.1, 100.0)
- moved REF** 6.88 mm to (141.4, 90.2)
- moved REF** 6.88 mm to (177.8, 129.5)
- moved ? 6.88 mm to (282.3, 107.2)
- moved REF** 6.88 mm to (163.3, 169.4)
- moved REF** 6.88 mm to (290.7, 71.8)
- moved REF** 6.88 mm to (271.7, 136.7)
- moved REF** 6.88 mm to (180.6, 180.3)
- moved REF** 6.88 mm to (231.6, 201.9)
- moved REF** 6.88 mm to (283.9, 111.6)
- moved REF** 6.88 mm to (212.8, 156.5)
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Routing:
- net (no net): track 4177.6 -> 5286.7 mm
Other:
- outline, holes or cut-outs redrawn
- board text added: "섴"

Commit message: Completes row/col silkscreen for seok-38_Mk1_rev0
Parts:
- moved REF** 15.2 mm to (229.2, 129.8)
- renumbered REF** to D0:0, REF** to D0:1, REF** to D0:2, REF** to D0:3, REF** to D0:4, REF** to D0:5, REF** to D0:6, REF** to D0:7, REF** to D0:8, REF** to D0:9, REF** to D1:0, REF** to D1:1, REF** to D1:2, REF** to D1:3, REF** to D1:4, REF** to D1:5, REF** to D1:6, REF** to D1:7, REF** to D1:8, REF** to D1:9, REF** to D2:0, REF** to D2:1, REF** to D2:2, REF** to D2:3, REF** to D2:4, REF** to D2:5, REF** to D2:6, REF** to D2:8, REF** to D2:9, REF** to D3:0, REF** to D3:2, REF** to D3:3, REF** to D3:4, REF** to D3:5, REF** to D3:6, REF** to D3:9, REF** to H0, REF** to H1, REF** to H2, REF** to H3, REF** to H4, REF** to S0:0, REF** to S0:1, REF** to S0:2, REF** to S0:3, REF** to S0:4, REF** to S0:5, REF** to S0:6, REF** to S0:7, REF** to S0:8, REF** to S0:9, REF** to S1:0, REF** to S1:1, REF** to S1:2, REF** to S1:3, REF** to S1:4, REF** to S1:5, REF** to S1:6, REF** to S1:7, REF** to S1:8, REF** to S1:9, REF** to S2:0, REF** to S2:1, REF** to S2:2, REF** to S2:3, REF** to S2:4, REF** to S2:5, REF** to S2:6, REF** to S2:7, REF** to S2:8, REF** to S2:9, REF** to S3:0, REF** to S3:2, REF** to S3:3, REF** to S3:4, REF** to S3:5, REF** to S3:6, REF** to S3:7, REF** to S3:9
Routing:
- net (no net): track 5286.7 -> 5253.6 mm
Other:
- board text added: "-38"
- board text added: "SEOK"
- board text added: "Split Ergonomic Ortholinear Keyboard"

Commit message: Add final silkscreen labelling to seok-38_Mk1_rev0
Parts:
- renumbered REF** to RESET
Routing:
- net (no net): track 5253.6 -> 5281.5 mm
Other:
- outline, holes or cut-outs redrawn
- board text added: "01-2024"
- board text added: "C0"
- board text added: "C1"
- board text added: "C2"
- board text added: "C3"
- board text added: "C4"
- board text added: "C5"
- board text added: "C6"
- board text added: "C7"
- board text added: "C8"
- board text added: "C9"
- board text added: "GND"
- board text added: "HAMLUND MFG."
- board text added: "I2C0"
- board text added: "Raspberry Pi Pico"
- board text added: "SCL"
- board text added: "SDA"
- board text added: "SEOK-38-MK.1-REV.0-M"
- board text added: "SSD1306 OLED 128x64"
- board text added: "VCC"
