File: kicad/seok-38/seok-38_Mk1_rev0/seok-38_Mk1_rev0.kicad_pcb (KiCad board)
At the start: 2 copper layers, 294.1 x 158 mm, 88 parts

Commit message: DRC and silkscreen updates
Parts:
- removed ? (x4): , 
- moved S3:0 25.0 mm to (75.4, 124.1)
- moved RESET 25.0 mm to (222.5, 153.9)
- moved S0:1 25.0 mm to (125.0, 104.9)
- moved S3:2 25.0 mm to (156.5, 193.5)
- moved S3:6 25.0 mm to (238.5, 205.1)
- moved S2:8 25.0 mm to (300.9, 142.5)
- moved D1:3 25.0 mm to (150.1, 130.5)
- moved S2:0 25.0 mm to (87.3, 149.7)
- moved D2:4 25.0 mm to (160.3, 160.9)
- moved REF** 25.0 mm to (206.1, 180.6)
- moved S0:2 25.0 mm to (145.5, 107.0)
- moved S1:4 25.0 mm to (171.1, 153.6)
- moved D2:6 25.0 mm to (261.7, 151.9)
- moved D1:1 25.0 mm to (114.2, 112.1)
- moved D3:6 25.0 mm to (235.3, 196.1)
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Other:
- board text added: "JLCJLCJLCJLC"
- board text added: "함룬드 제조"

Commit message: Final silkscreen and DRC tweaks before manufacturing
Parts:
- moved D1:8 15.2 mm to (296.6, 100.7)
- moved S0:8 15.2 mm to (293.0, 90.8)
- moved S1:6 15.2 mm to (263.9, 128.0)
- moved S1:8 15.2 mm to (299.8, 109.6)
- moved S3:9 15.2 mm to (342.5, 110.0)
- moved D0:4 15.2 mm to (179.8, 109.2)
- moved D0:5 15.2 mm to (236.8, 111.8)
- moved D0:6 15.2 mm to (253.8, 100.3)
- moved D1:0 15.2 mm to (96.0, 105.3)
- moved D1:4 15.2 mm to (172.9, 128.0)
- moved D1:5 15.2 mm to (243.6, 130.6)
- moved D1:6 15.2 mm to (260.7, 119.1)
- moved D2:0 15.2 mm to (89.2, 124.1)
- moved D2:4 15.2 mm to (166.1, 146.8)
- moved D2:5 15.2 mm to (250.4, 149.4)
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Other:
- board text added: "햄"
- board text added: "햄룬드 제조"
- board text removed: "함룬드 제조"

Commit message: Final final tweaks before manufacturing (lol)
Other:
- board text added: "Mk 1"
Changed lines of the file:
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@@
       (plot_on_all_layers_selection 0x0000000_00000000)
       (disableapertmacros false)
-      (usegerberextensions false)
-      (usegerberattributes true)
-      (usegerberadvancedattributes true)
-      (creategerberjobfile true)
+      (usegerberextensions true)
+      (usegerberattributes false)
+      (usegerberadvancedattributes false)
+      (creategerberjobfile false)
       (dashed_line_dash_ratio 12.000000)
       (dashed_line_gap_ratio 3.000000)
@@
       (psa4output false)
       (plotreference true)
-      (plotvalue true)
+      (plotvalue false)
       (plotinvisibletext false)
       (sketchpadsonfab false)
-      (subtractmaskfromsilk false)
+      (subtractmaskfromsilk true)
       (outputformat 1)
       (mirror false)
-      (drillshape 1)
+      (drillshape 0)
       (scaleselection 1)
-      (outputdirectory "")
+      (outputdirectory "C:/Users/shudock/Desktop/seok-38-fab-files-rev0/")
     )
   )
@@
     )
   )
+  (gr_text "Mk 1" (at 190.25 144.2 70) (layer "F.SilkS")
+    (effects (font (size 2 2) (thickness 0.32)) (justify left bottom))
+  )
   (gr_text "SSD1306\nOLED 128x64" (at 211.82696 181.562262) (layer "F.SilkS")
