File: kicad/mskp/io_ctrl_board_secondary_Mk1_rev0/io_ctrl_board_seconday_Mk1_rev0.kicad_sch (KiCad schematic)
At the start: 5 parts, among them J10 OLED_128x64, J4 USB_C_Receptacle_USB2.0, J5 Conn_01x04_Socket, J8 Conn_01x12_Socket, U2 MCP23017_SP

Commit message: Removes the mksp_Mk1_rev0 project in favor of board-specific projects
Parts:
- removed J5: Conn_01x04_Socket, symbol Connector:Conn_01x04_Socket
Changed lines of the file:
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@@
+        )
+      )
+      (project "peripheral-ctrl-board"
+        (path "/d92793f5-7a37-47c1-ba13-f28d416cb7ec"
+          (reference "J8") (unit 1)
         )
       )
@@
         (path "/317db825-7ec8-42a4-86c9-29de77488848/6eeaa44f-3e3d-4d86-815d-42d0f349cb86"
           (reference "J3") (unit 1)
+        )
+      )
+      (project "peripheral-ctrl-board"
+        (path "/d92793f5-7a37-47c1-ba13-f28d416cb7ec"
+          (reference "J4") (unit 1)
         )
       )
@@
         )
       )
+      (project "peripheral-ctrl-board"
+        (path "/d92793f5-7a37-47c1-ba13-f28d416cb7ec"
+          (reference "U2") (unit 1)
+        )
+      )
     )
   )
@@
         )
       )
-    )
-  )
-  (symbol (lib_id "Connector:Conn_01x04_Socket") (at 236.22 50.8 0) (unit 1)
-    (in_bom yes) (on_board yes) (dnp no) (fields_autoplaced)
-    (property "Reference" "J5" (at 237.49 50.8 0)
-      (effects (font (size 1.27 1.27)) (justify left))
-    )
-    (property "Value" "Conn_01x04_Socket" (at 237.49 53.34 0)
-      (effects (font (size 1.27 1.27)) (justify left))
-    )
-    (property "Footprint" "" (at 236.22 50.8 0)
-      (effects (font (size 1.27 1.27)) hide)
-    )
-    (property "Datasheet" "~" (at 236.22 50.8 0)
-      (effects (font (size 1.27 1.27)) hide)
-    )
-    (pin "1")
-    (pin "2")
-    (pin "3")
-    (pin "4")
-    (instances
-      (project "mksp_Mk1_rev0"
-        (path "/317db825-7ec8-42a4-86c9-29de77488848/9a4d8874-164c-4918-b768-ce32cb89a53f"
-          (reference "J5") (unit 1)
-        )
-        (path "/317db825-7ec8-42a4-86c9-29de77488848/6eeaa44f-3e3d-4d86-815d-42d0f349cb86"
-          (reference "J6") (unit 1)
+      (project "peripheral-ctrl-board"
+        (path "/d92793f5-7a37-47c1-ba13-f28d416cb7ec"
+          (reference "J10") (unit 1)
         )
       )
     )
   )
+  (sheet_instances
+    (path "/" (page "1"))
+  )
 )
