File: kicad/mskp/seok-42_mx_keypad_L_Mk1_rev0/seok-42_mx_keypad_L_Mk1_rev0.kicad_sch (KiCad schematic)
At the start: 43 parts, among them J1 Conn_01x12_Socket, SW1 Switch, SW10 Switch, SW11 Switch, SW12 Switch, SW13 Switch, SW14 Switch, SW15 Switch, SW16 Switch, SW17 Switch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

Commit message: Initial work on seok-42_mx_keypad_L_Mk1_rev0 layout
Parts:
- J1: footprint (none) -> Connector_JST:JST_GH_SM12B-GHS-TB_1x12-1MP_P1.25mm_Horizontal
- SW1, SW10, SW11, SW12, SW13, SW14, SW15, SW16, SW17, SW18, SW19, SW2, SW20, SW21, SW3, SW4, SW5, SW6, SW7, SW8, SW9: footprint (none) -> ScottoKeebs_Hotswap:Hotswap_MX_Plated_1.00u
Connections:
- net at SW11.2, SW18.2, SW4.2: now also J1.9 (Pin_9)
- net at D12.1 (K): now also D10.1 (K), D11.1 (K), D13.1 (K), D14.1 (K), D8.1 (K), D9.1 (K), J1.2 (Pin_2)
- net at D3.1 (K): now also D1.1 (K), D2.1 (K), D4.1 (K), D5.1 (K), D6.1 (K), D7.1 (K), J1.1 (Pin_1)
- net at SW1.2, SW15.2, SW8.2: now also J1.12 (Pin_12)
- net at SW16.1: now also D16.2 (A)
- net at SW16.2, SW2.2, SW9.2: now also J1.11 (Pin_11)
- net at SW13.2, SW20.2, SW6.2: now also J1.7 (Pin_7)
- net at SW12.2, SW19.2, SW5.2: now also J1.8 (Pin_8)
- net at D20.1 (K): now also D15.1 (K), D16.1 (K), D17.1 (K), D18.1 (K), D19.1 (K), D21.1 (K), J1.3 (Pin_3)
- net at J1.10 (Pin_10): now also SW10.2, SW17.2, SW3.2
- net at J1.6 (Pin_6): now also SW14.2, SW21.2, SW7.2
- no-connect marks 0 -> 2
