File: kicad/mskp/pico_ctrl_board_primary_Mk2_rev0/pico_ctrl_board_primary_Mk2_rev0.kicad_pcb (KiCad board)
At the start: 2 copper layers, 51.2 x 71.5 mm, 29 parts, among them J1 USB_C_I2C_Receptacle, J10 Conn_01x02_Socket, J2 SPI-JST, J3 RJ45_I2C_SPI_Port, J4 UART-JST, J5 I2C-aux-pad, J6 OLED_128x64, J7 Keypad-Matrix_JST, J8 USB_sw_ctrl, J9 Debug_pads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

Commit message: Final tweaks to PCBs before second round of mskp fabrications
Routing:
- net +5V: track 159.8 -> 158.1 mm
Other:
- board text added: "github.com/"
- board text added: "thegreatgramblinham"
- board text removed: "github.com/thegreatgramblinham"
Changed lines of the file:
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@@
 			(plot_on_all_layers_selection 0x0000000_00000000)
 			(disableapertmacros no)
-			(usegerberextensions no)
-			(usegerberattributes yes)
-			(usegerberadvancedattributes yes)
-			(creategerberjobfile yes)
+			(usegerberextensions yes)
+			(usegerberattributes no)
+			(usegerberadvancedattributes no)
+			(creategerberjobfile no)
 			(dashed_line_dash_ratio 12.000000)
 			(dashed_line_gap_ratio 3.000000)
 			(svgprecision 4)
 			(plotframeref no)
-			(viasonmask no)
+			(viasonmask yes)
 			(mode 1)
 			(useauxorigin no)
@@
 			(psa4output no)
 			(plotreference yes)
-			(plotvalue yes)
+			(plotvalue no)
 			(plotfptext yes)
 			(plotinvisibletext no)
 			(sketchpadsonfab no)
-			(subtractmaskfromsilk no)
+			(subtractmaskfromsilk yes)
 			(outputformat 1)
 			(mirror no)
-			(drillshape 1)
+			(drillshape 0)
 			(scaleselection 1)
-			(outputdirectory "")
+			(outputdirectory "pico_ctrl_mk2_exports")
 		)
 	)
@@
 		)
 	)
+	(gr_text "thegreatgramblinham"
+		(at 142.7 83.9 0)
+		(layer "F.SilkS")
+		(effects
+			(font
+				(size 1 1)
+				(thickness 0.1)
+				(italic yes)
+			)
+			(justify left bottom)
+		)
+	)
 	(gr_text "I2C"
 		(at 113.95 110.35 0)
@@
 		)
 	)
-	(gr_text "github.com/thegreatgramblinham"
-		(at 116.8 73.85 90)
+	(gr_text "github.com/"
+		(at 141.7 82.4 0)
 		(layer "F.SilkS")
 		(effects
@@
 				(size 1 1)
 				(thickness 0.1)
+				(italic yes)
 			)
 			(justify left bottom)
@@
 	)
 	(gr_text "JLCJLCJLCJLC"
-		(at 127.4 115.4 0)
+		(at 141.9 89.3 0)
 		(layer "F.SilkS")
 		(effects
@@
 	)
 	(segment
-		(start 147.7 91.05)
-		(end 148.15 91.5)
-		(width 0.5)
-		(layer "F.Cu")
-		(net 3)
-	)
-	(segment
-		(start 141.15 104.95)
-		(end 136.15 104.95)
+		(start 143.75 52.1875)
+		(end 141.8125 52.1875)
 		(width 0.5)
 		(layer "F.Cu")
@@
 	)
 	(segment
-		(start 143.75 52.1875)
-		(end 141.8125 52.1875)
+		(start 146.65 93.25)
+		(end 153.62 93.25)
 		(width 0.5)
 		(layer "F.Cu")
@@
 	)
 	(segment
-		(start 148.15 91.5)
-		(end 148.15 93.25)
+		(start 146.415 78.835)
+		(end 143.5 81.75)
 		(width 0.5)
 		(layer "F.Cu")
@@
 	)
 	(segment
-		(start 136.15 104.95)
-		(end 135.1 106)
+		(start 116.85 48.15)
+		(end 136.17 48.15)
 		(width 0.5)
 		(layer "F.Cu")
@@
 	)
 	(segment
-		(start 143.5 81.75)
-		(end 143.5 88.85)
+		(start 145.9 95.45)
+		(end 141.5 99.85)
 		(width 0.5)
 		(layer "F.Cu")
@@
 	)
 	(segment
-		(start 116.85 48.15)
-		(end 136.17 48.15)
+		(start 135.1 108.85)
+		(end 134.3875 109.5625)
 		(width 0.5)
 		(layer "F.Cu")
@@
 	)
 	(segment
-		(start 134.3875 109.5625)
-		(end 129.5 109.5625)
+		(start 141.865 49.87)
+		(end 143.735 48)
 		(width 0.5)
 		(layer "F.Cu")
@@
 	)
 	(segment
-		(start 141.865 49.87)
-		(end 143.735 48)
+		(start 145.9 92.5)
+		(end 146.65 93.25)
 		(width 0.5)
 		(layer "F.Cu")
@@
 	)
 	(segment
-		(start 145.9 95.45)
-		(end 145.525 95.825)
+		(start 145.9 91.25)
+		(end 145.9 95.45)
 		(width 0.5)
 		(layer "F.Cu")
@@
 	)
 	(segment
-		(start 135.1 108.85)
-		(end 134.3875 109.5625)
-		(width 0.5)
-		(layer "F.Cu")
-		(net 3)
-	)
-	(segment
 		(start 114.8125 56.8125)
 		(end 115.55 57.55)
@@
 	)
 	(segment
-		(start 143.5 88.85)
-		(end 145.7 91.05)
-		(width 0.5)
-		(layer "F.Cu")
-		(net 3)
-	)
-	(segment
 		(start 115.55 57.55)
 		(end 115.55 59.65)
@@
 	)
 	(segment
-		(start 129.5 109.5625)
-		(end 127.8925 109.5625)
+		(start 135.1 106)
+		(end 135.1 108.85)
 		(width 0.5)
 		(layer "F.Cu")
@@
 	)
 	(segment
-		(start 135.1 106)
-		(end 135.1 108.85)
+		(start 141.5 99.85)
+		(end 141.5 104.6)
 		(width 0.5)
 		(layer "F.Cu")
@@
 	)
 	(segment
-		(start 148.15 93.25)
-		(end 153.62 93.25)
+		(start 129.5 109.5625)
+		(end 127.8925 109.5625)
 		(width 0.5)
 		(layer "F.Cu")
@@
 	)
 	(segment
-		(start 146.415 77.75)
-		(end 146.415 78.835)
+		(start 136.15 104.95)
+		(end 135.1 106)
 		(width 0.5)
 		(layer "F.Cu")
@@
 	)
 	(segment
-		(start 146.415 78.835)
-		(end 143.5 81.75)
-		(width 0.5)
-		(layer "F.Cu")
-		(net 3)
-	)
-	(segment
-		(start 145.9 91.05)
-		(end 145.9 95.45)
+		(start 146.415 77.75)
+		(end 146.415 78.835)
 		(width 0.5)
 		(layer "F.Cu")
@@
 	)
 	(segment
-		(start 146.465 77.8)
-		(end 146.415 77.75)
+		(start 134.3875 109.5625)
+		(end 129.5 109.5625)
 		(width 0.5)
 		(layer "F.Cu")
@@
 	)
 	(segment
-		(start 145.7 91.05)
-		(end 145.9 91.05)
+		(start 143.5 81.75)
+		(end 143.5 88.85)
 		(width 0.5)
 		(layer "F.Cu")
@@
 	)
 	(segment
-		(start 127.8925 109.5625)
-		(end 125.58 107.25)
+		(start 143.5 88.85)
+		(end 145.9 91.25)
 		(width 0.5)
 		(layer "F.Cu")
@@
 	)
 	(segment
-		(start 141.5 104.6)
-		(end 141.15 104.95)
+		(start 146.465 77.8)
+		(end 146.415 77.75)
 		(width 0.5)
 		(layer "F.Cu")
@@
 	)
 	(segment
-		(start 114.8125 55)
-		(end 114.8125 52.1875)
+		(start 127.8925 109.5625)
+		(end 125.58 107.25)
 		(width 0.5)
 		(layer "F.Cu")
@@
 	)
 	(segment
-		(start 145.525 95.825)
-		(end 141.5 99.85)
+		(start 141.15 104.95)
+		(end 136.15 104.95)
 		(width 0.5)
 		(layer "F.Cu")
@@
 	)
 	(segment
-		(start 115.85 51.15)
-		(end 115.85 49.15)
+		(start 114.8125 55)
+		(end 114.8125 52.1875)
 		(width 0.5)
 		(layer "F.Cu")
@@
 	)
 	(segment
-		(start 141.5 99.85)
-		(end 141.5 104.6)
+		(start 115.85 51.15)
+		(end 115.85 49.15)
 		(width 0.5)
 		(layer "F.Cu")
@@
 	)
 	(segment
-		(start 145.9 91.05)
-		(end 147.7 91.05)
+		(start 146.9 52.2)
+		(end 143.7625 52.2)
 		(width 0.5)
 		(layer "F.Cu")
@@
 	)
 	(segment
-		(start 146.9 52.2)
-		(end 143.7625 52.2)
+		(start 137.89 52.41)
+		(end 137.89 49.87)
 		(width 0.5)
 		(layer "F.Cu")
@@
 	)
 	(segment
-		(start 137.89 52.41)
-		(end 137.89 49.87)
+		(start 141.5 104.6)
+		(end 141.15 104.95)
 		(width 0.5)
 		(layer "F.Cu")
@@
 		(net 9)
 	)
-	(segment
-		(start 133.955026 100.494974)
-		(end 133.9 100.439949)
-		(width 0.15)
-		(layer "B.Cu")
-		(net 9)
-	)
